File: ESP_DIP_MIN.sch (KiCad schematic (older format))
At the start: 7 parts, among them U1 ESP32-WROOM

Commit message: initial commit
Parts:
- removed I2C1: Conn_01x02_Male, symbol Connector:Conn_01x02_Male
- removed IO_LED1: Conn_01x01_Male, symbol Connector:Conn_01x01_Male
- removed SPI1: Conn_01x05_Male, symbol Connector:Conn_01x05_Male
- added COMM1: Conn_01x08_Male, Connector_PinHeader_2.54mm:PinHeader_1x08_P2.54mm_Vertical, symbol Connector:Conn_01x08_Male
- added J1, J2, J3, J4: Conn_01x01_Male, MountingHole:MountingHole_3.2mm_M3, symbol Connector:Conn_01x01_Male
- POWER1, UART1: footprint (none) -> Connector_PinHeader_2.54mm:PinHeader_1x02_P2.54mm_Vertical
- SWITCH1: renamed from UART2; footprint (none) -> Connector_PinHeader_2.54mm:PinHeader_1x02_P2.54mm_Vertical
Connections:
- net labels added: SCK
Changed lines of the file:
@@
 F 0 "POWER1" H 5356 1578 50  0000 C CNN
 F 1 "Conn_01x02_Male" H 5356 1487 50  0000 C CNN
-F 2 "" H 5250 1400 50  0001 C CNN
+F 2 "Connector_PinHeader_2.54mm:PinHeader_1x02_P2.54mm_Vertical" H 5250 1400 50  0001 C CNN
 F 3 "~" H 5250 1400 50  0001 C CNN
 	1    5250 1400
 	1    0    0    -1
 $EndComp
-$Comp
-L Connector:Conn_01x02_Male I2C1
-U 1 1 5BC5ABBD
-P 5250 2000
-F 0 "I2C1" H 5356 2178 50  0000 C CNN
-F 1 "Conn_01x02_Male" H 5356 2087 50  0000 C CNN
-F 2 "" H 5250 2000 50  0001 C CNN
-F 3 "~" H 5250 2000 50  0001 C CNN
-	1    5250 2000
-	1    0    0    -1
-$EndComp
-$Comp
-L Connector:Conn_01x01_Male IO_LED1
-U 1 1 5BC5ACE8
-P 5250 3100
-F 0 "IO_LED1" H 5356 3278 50  0000 C CNN
-F 1 "Conn_01x01_Male" H 5356 3187 50  0000 C CNN
-F 2 "" H 5250 3100 50  0001 C CNN
-F 3 "~" H 5250 3100 50  0001 C CNN
-	1    5250 3100
-	1    0    0    -1
-$EndComp
-Text GLabel 5750 2000 2    50   Input ~ 0
+Text GLabel 5800 2700 2    50   Input ~ 0
 SCL
-Text GLabel 5750 2100 2    50   Input ~ 0
+Text GLabel 5800 2800 2    50   Input ~ 0
 SDA
-Text GLabel 5750 3100 2    50   Input ~ 0
+Text GLabel 5800 2100 2    50   Input ~ 0
 IO_LED
 Text GLabel 5750 1400 2    50   Input ~ 0
@@
 	4100 3050 4400 3050
 Wire Wire Line
-	5450 2000 5750 2000
-Wire Wire Line
-	5750 2100 5450 2100
-Wire Wire Line
-	5450 3100 5750 3100
+	5500 2100 5800 2100
+Wire Wire Line
+	5800 2200 5500 2200
+Wire Wire Line
+	5500 2800 5800 2800
 $Comp
 L power:GND #PWR01
@@
 Wire Wire Line
 	4100 2750 4400 2750
-Text GLabel 5750 2400 2    50   Input ~ 0
+Text GLabel 5800 2400 2    50   Input ~ 0
 D3
-Text GLabel 5750 2500 2    50   Input ~ 0
+Text GLabel 5800 2500 2    50   Input ~ 0
 CMD
-Text GLabel 5750 2600 2    50   Input ~ 0
-CLK
-Text GLabel 5750 2700 2    50   Input ~ 0
+Text GLabel 5800 2300 2    50   Input ~ 0
+SCK
+Text GLabel 5800 2600 2    50   Input ~ 0
 D0
 Wire Wire Line
-	5450 2400 5750 2400
-Wire Wire Line
-	5450 2500 5750 2500
-Wire Wire Line
-	5450 2600 5750 2600
-Wire Wire Line
-	5450 2700 5750 2700
-Text GLabel 5750 2800 2    50   Input ~ 0
+	5500 2300 5800 2300
+Wire Wire Line
+	5500 2400 5800 2400
+Wire Wire Line
+	5500 2500 5800 2500
+Wire Wire Line
+	5500 2600 5800 2600
+Text GLabel 5800 2200 2    50   Input ~ 0
 CD
-$Comp
-L Connector:Conn_01x05_Male SPI1
-U 1 1 5BC5D8EE
-P 5250 2600
-F 0 "SPI1" H 5356 2978 50  0000 C CNN
-F 1 "Conn_01x05_Male" H 5356 2887 50  0000 C CNN
-F 2 "" H 5250 2600 50  0001 C CNN
-F 3 "~" H 5250 2600 50  0001 C CNN
-	1    5250 2600
-	1    0    0    -1
-$EndComp
-Wire Wire Line
-	5450 2800 5750 2800
 Text GLabel 4400 1850 2    50   Input ~ 0
 TXD
@@
 F 0 "UART1" H 5356 3578 50  0000 C CNN
 F 1 "Conn_01x02_Male" H 5356 3487 50  0000 C CNN
-F 2 "" H 5250 3400 50  0001 C CNN
+F 2 "Connector_PinHeader_2.54mm:PinHeader_1x02_P2.54mm_Vertical" H 5250 3400 50  0001 C CNN
 F 3 "~" H 5250 3400 50  0001 C CNN
 	1    5250 3400
@@
 CMD
 Text GLabel 6450 2600 0    50   Input ~ 0
-CLK
+SCK
 Text GLabel 6450 2700 0    50   Input ~ 0
 D0
@@
 $EndComp
 $Comp
-L Connector:Conn_01x02_Male UART2
+L Connector:Conn_01x02_Male SWITCH1
 U 1 1 5BCB6DBB
 P 5250 3800
-F 0 "UART2" H 5356 3978 50  0000 C CNN
+F 0 "SWITCH1" H 5356 3978 50  0000 C CNN
 F 1 "Conn_01x02_Male" H 5356 3887 50  0000 C CNN
-F 2 "" H 5250 3800 50  0001 C CNN
+F 2 "Connector_PinHeader_2.54mm:PinHeader_1x02_P2.54mm_Vertical" H 5250 3800 50  0001 C CNN
 F 3 "~" H 5250 3800 50  0001 C CNN
 	1    5250 3800
@@
 Wire Wire Line
 	5750 3900 5450 3900
+Wire Wire Line
+	5500 2700 5800 2700
+$Comp
+L Connector:Conn_01x08_Male COMM1
+U 1 1 5BC66FA9
+P 5300 2400
+F 0 "COMM1" H 5406 2878 50  0000 C CNN
+F 1 "Conn_01x08_Male" H 5406 2787 50  0000 C CNN
+F 2 "Connector_PinHeader_2.54mm:PinHeader_1x08_P2.54mm_Vertical" H 5300 2400 50  0001 C CNN
+F 3 "~" H 5300 2400 50  0001 C CNN
+	1    5300 2400
+	1    0    0    -1
+$EndComp
+$Comp
+L Connector:Conn_01x01_Male J1
+U 1 1 5BC6C17B
+P 2000 4300
+F 0 "J1" H 2106 4478 50  0000 C CNN
+F 1 "Conn_01x01_Male" H 2106 4387 50  0000 C CNN
+F 2 "MountingHole:MountingHole_3.2mm_M3" H 2000 4300 50  0001 C CNN
+F 3 "~" H 2000 4300 50  0001 C CNN
+	1    2000 4300
+	1    0    0    -1
+$EndComp
+$Comp
+L Connector:Conn_01x01_Male J2
+U 1 1 5BC6C1B7
+P 2000 4500
+F 0 "J2" H 2106 4678 50  0000 C CNN
+F 1 "Conn_01x01_Male" H 2106 4587 50  0000 C CNN
+F 2 "MountingHole:MountingHole_3.2mm_M3" H 2000 4500 50  0001 C CNN
+F 3 "~" H 2000 4500 50  0001 C CNN
+	1    2000 4500
+	1    0    0    -1
+$EndComp
+$Comp
+L Connector:Conn_01x01_Male J3
+U 1 1 5BC6C1DD
+P 2000 4700
+F 0 "J3" H 2106 4878 50  0000 C CNN
+F 1 "Conn_01x01_Male" H 2106 4787 50  0000 C CNN
+F 2 "MountingHole:MountingHole_3.2mm_M3" H 2000 4700 50  0001 C CNN
+F 3 "~" H 2000 4700 50  0001 C CNN
+	1    2000 4700
+	1    0    0    -1
+$EndComp
+$Comp
+L Connector:Conn_01x01_Male J4
+U 1 1 5BC6C205
+P 2000 4900
+F 0 "J4" H 2106 5078 50  0000 C CNN
+F 1 "Conn_01x01_Male" H 2106 4987 50  0000 C CNN
+F 2 "MountingHole:MountingHole_3.2mm_M3" H 2000 4900 50  0001 C CNN
+F 3 "~" H 2000 4900 50  0001 C CNN
+	1    2000 4900
+	1    0    0    -1
+$EndComp
 $EndSCHEMATC

Commit message: resolve mistake
Parts:
- added R1: 5.1k, symbol Device:R
- added R?: 10k, symbol Device:R
Connections:
- net labels removed: CLK, CMD, D0, D3
- no-connect marks 22 -> 21
Changed lines of the file:
@@
 Wire Wire Line
 	4100 2750 4400 2750
-Text GLabel 5800 2400 2    50   Input ~ 0
-D3
-Text GLabel 5800 2500 2    50   Input ~ 0
-CMD
-Text GLabel 5800 2300 2    50   Input ~ 0
-SCK
-Text GLabel 5800 2600 2    50   Input ~ 0
-D0
 Wire Wire Line
 	5500 2300 5800 2300
@@
 MISO
 Text GLabel 4400 2350 2    50   Input ~ 0
-CLK
+SCK
 Text GLabel 4400 2450 2    50   Input ~ 0
 CS
-Text GLabel 4400 2550 2    50   Input ~ 0
+Text GLabel 4400 1650 2    50   Input ~ 0
 MOSI
 Wire Wire Line
@@
 Wire Wire Line
 	4100 2450 4400 2450
-Wire Wire Line
-	4100 2550 4400 2550
 Text GLabel 4400 2650 2    50   Input ~ 0
 CD
 Wire Wire Line
 	4100 2650 4400 2650
-Text GLabel 6950 2400 2    50   Input ~ 0
-CS
-Text GLabel 6950 2500 2    50   Input ~ 0
-CLK
-Text GLabel 6950 2600 2    50   Input ~ 0
-MOSI
-Text GLabel 6950 2700 2    50   Input ~ 0
-MISO
-Text GLabel 6450 2400 0    50   Input ~ 0
-D3
-Text GLabel 6450 2500 0    50   Input ~ 0
-CMD
-Text GLabel 6450 2600 0    50   Input ~ 0
-SCK
-Text GLabel 6450 2700 0    50   Input ~ 0
-D0
-Wire Wire Line
-	6450 2400 6950 2400
-Wire Wire Line
-	6950 2500 6450 2500
-Wire Wire Line
-	6450 2600 6950 2600
-Wire Wire Line
-	6950 2700 6450 2700
 Text GLabel 4400 2850 2    50   Input ~ 0
 BOOT
 Wire Wire Line
 	4100 2850 4400 2850
-NoConn ~ 4100 1650
 NoConn ~ 4100 2950
 NoConn ~ 2250 3000
@@
 NoConn ~ 3450 3450
 NoConn ~ 3550 3450
-NoConn ~ 3650 3450
 $Comp
 L power:PWR_FLAG #FLG01
@@
 	1    0    0    -1
 $EndComp
+$Comp
+L Device:R R1
+U 1 1 5BC82C7C
+P 3650 3600
+F 0 "R1" H 3720 3646 50  0000 L CNN
+F 1 "5.1k" H 3720 3555 50  0000 L CNN
+F 2 "" V 3580 3600 50  0001 C CNN
+F 3 "~" H 3650 3600 50  0001 C CNN
+	1    3650 3600
+	1    0    0    -1
+$EndComp
+$Comp
+L power:GND #PWR0101
+U 1 1 5BC82D6F
+P 3650 3900
+F 0 "#PWR0101" H 3650 3650 50  0001 C CNN
+F 1 "GND" H 3655 3727 50  0000 C CNN
+F 2 "" H 3650 3900 50  0001 C CNN
+F 3 "" H 3650 3900 50  0001 C CNN
+	1    3650 3900
+	1    0    0    -1
+$EndComp
+Wire Wire Line
+	3650 3750 3650 3900
+NoConn ~ 4400 2550
+Wire Wire Line
+	4100 2550 4400 2550
+Text GLabel 5800 2600 2    50   Input ~ 0
+CS
+Text GLabel 5800 2500 2    50   Input ~ 0
+SCK
+Wire Wire Line
+	4100 1650 4400 1650
+Text GLabel 5800 2400 2    50   Input ~ 0
+MISO
+Text GLabel 5800 2300 2    50   Input ~ 0
+MOSI
+Text GLabel 7100 2450 2    50   Input ~ 0
+MISO
+Text GLabel 6500 2450 0    50   Input ~ 0
+VCC
+$Comp
+L Device:R R?
+U 1 1 5BC8E4FB
+P 6800 2450
+F 0 "R?" V 6593 2450 50  0000 C CNN
+F 1 "10k" V 6684 2450 50  0000 C CNN
+F 2 "" V 6730 2450 50  0001 C CNN
+F 3 "~" H 6800 2450 50  0001 C CNN
+	1    6800 2450
+	0    1    1    0
+$EndComp
+Wire Wire Line
+	6500 2450 6650 2450
+Wire Wire Line
+	6950 2450 7100 2450
 $EndSCHEMATC
